Commit message: rebuilt the hdt urdfs using our stls and inertias, and giving intuitive names to the links

File: urdf/hdt_7dof_left.xacro (robot description, xacro)
@@ -9,4 +9,4 @@
 	<link name="world" />
 	<xacro:include filename="$(find hdt_7dof_description)/urdf/hdt_7dof_left_macro.xacro" />
-	<xacro:hdt_7dof_left parent="world" x="0" y="0" z="0" yaw="-1.57079" prefix="left_" />
+	<xacro:hdt_7dof_left parent="world" x="0" y="0" z="0" prefix="left_" />
 </robot>

File: urdf/hdt_7dof_left_macro.xacro (robot description, xacro)
@@ -8,28 +8,28 @@
 		izz="0.0005"/>
 	</xacro:macro>
-	<xacro:macro name="hdt_7dof_left" params="parent x y z yaw prefix">
+	<xacro:macro name="hdt_7dof_left" params="parent x y z prefix">
 		<!-- materials -->
 		<material name="${prefix}green">
-			<color rgba="${53/255} ${94/255} ${59/255} 1.0"/>
+			<color rgba="0.2078431372549 0.36862745098039 0.23137254901961 1.0"/>
 		</material>
 		<material name="${prefix}black">
-			<color rgba="${0/255} ${0/255} ${0/255} 1.0"/>
+			<color rgba="0 0 0 1.0"/>
 		</material>
 		<material name="${prefix}grey">
-			<color rgba="${40/255} ${40/255} ${40/255} 1.0"/>
+			<color rgba="0.15686274509804 0.15686274509804 0.15686274509804 1.0"/>
 		</material>
-		<!-- segment 1 -->
-		<joint name="${prefix}joint1" type="revolute">
+		<!-- shoulder-->
+		<joint name="${prefix}shoulder_pitch" type="revolute">
 			<hdt id="41" kmin="100" kmax="200" inertia="0.1"/>
-			<axis xyz="-1 0 0"/>
-			<limit effort="60.0" lower="-3.1416" upper="1.0472" velocity="2.0944"/>
-			<origin xyz="${x} ${y} ${z}" rpy="0 0 ${yaw}"/>
+			<axis xyz="0 1 0"/>
+			<limit effort="60.0" lower="-3.1415926535898" upper="1.0471975511966" velocity="2.0944"/>
+			<origin xyz="${x} ${y} ${z}" rpy="0 0 0"/>
 			<parent link="${parent}"/>
-			<child link="${prefix}link1"/>
+			<child link="${prefix}shoulder"/>
 			<dynamics damping="0.7" friction="0.0"/>
 		</joint>
 		<transmission name="${prefix}tran1">
 			<type>transmission_interface/SimpleTransmission</type>
-			<joint name="${prefix}joint1">
+			<joint name="${prefix}shoulder_pitch">
 				<hardwareInterface>EffortJointInterface</hardwareInterface>
 			</joint>
@@ -38,74 +38,43 @@
 			</actuator>
 		</transmission>
-		<link name="${prefix}link1">
-			<collision>
-				<origin xyz="0 0 0" rpy="0 0 0"/>
-				<geometry>
-					<mesh filename="package://hdt_7dof_description/meshes/hdt_7dof_1_right.STL"/>
-				</geometry>
-			</collision>
-			<visual>
-				<origin xyz="0 0 0" rpy="0 0 0"/>
-				<geometry>
-					<mesh filename="package://hdt_7dof_description/meshes/hdt_7dof_1_right.STL"/>
+		<link name="${prefix}shoulder">
+			<collision>
+				<origin xyz="-0.06 -0.134925 -1.04" rpy="0 0 0"/>
+				<geometry>
+					<mesh filename="package://hdt_7dof_description/meshes/ShoulderPitchLeft.stl" scale="0.001 0.001 0.001"/>
+				</geometry>
+			</collision>
+			<visual>
+				<origin xyz="-0.06 -0.134925 -1.04" rpy="0 0 0"/>
+				<geometry>
+					<mesh filename="package://hdt_7dof_description/meshes/ShoulderPitchLeft.stl" scale="0.001 0.001 0.001"/>
 				</geometry>
 				<material name="${prefix}green"/>
 			</visual>
 			<inertial>
-			<origin xyz="-0.04488 0 0" rpy="0 0 0"/>
-			<mass value="1.00775"/>
-				<inertia
-				ixx="0.00064952" ixy="0.0" ixz="0.0"
-				iyy="0.00104342" iyz="0.0"
-				izz="0.00104342"/>
-			</inertial>
-		</link>
-		<gazebo reference="${prefix}link1">
+				<origin xyz="0.000193283 -0.352347455 -0.00014774800000006" rpy="0 0 0"/>
+				<mass value="1.344398311"/>
+				<inertia
+				ixx="0.002733115" ixy="-7.2667e-05" ixz="1.21e-07"
+				iyy="0.001266353" iyz="1.541e-06"
+				izz="0.002795463"/>
+			</inertial>
+		</link>
+		<gazebo reference="${prefix}shoulder">
 			<material>Gazebo/Green</material>
 		</gazebo>
-		<joint name="${prefix}joint1f" type="fixed">
-			<parent link="${prefix}link1"/>
-			<child link="${prefix}link2a"/>
-			<origin xyz="-0.09217 0 0" rpy="0 0 0"/>
-		</joint>
-		<link name="${prefix}link2a">
-			<collision>
-				<origin xyz="0 0 0" rpy="0 0 0"/>
-				<geometry>
-					<mesh filename="package://hdt_7dof_description/meshes/hdt_7dof_2a_right.STL"/>
-				</geometry>
-			</collision>
-			<visual>
-				<origin xyz="0 0 0" rpy="0 0 0"/>
-				<geometry>
-					<mesh filename="package://hdt_7dof_description/meshes/hdt_7dof_2a_right.STL"/>
-				</geometry>
-				<material name="${prefix}black"/>
-			</visual>
-			<inertial>
-				<origin xyz="-0.04416876 0 0" rpy="0 0 0"/>
-				<mass value="0.66774822"/>
-				<inertia
-				ixx="0.00062987" ixy="0.0" ixz="0.0"
-				iyy="0.00091291" iyz="0.0"
-				izz="0.00110241"/>
-			</inertial>
-		</link>
-		<gazebo reference="${prefix}link2a">
-			<material>Gazebo/Black</material>
-		</gazebo>
-		<!-- segment 2 -->
-		<joint name="${prefix}joint2" type="revolute">
+		<!-- shoulder roll -->
+		<joint name="${prefix}shoulder_roll" type="revolute">
 			<hdt id="42" kmin="100" kmax="200" inertia="0.1"/>
-			<axis xyz="0 1 0"/>
-			<limit effort="60.0" lower="-0.5236" upper="3.1416" velocity="2.0944"/>
-			<origin xyz="-0.07 0 0" rpy="0 0 0"/>
-			<parent link="${prefix}link2a"/>
-			<child link="${prefix}link2b"/>
+			<axis xyz="1 0 0"/>
+			<limit effort="60.0" lower="-0.5235987755983" upper="3.1415926535898" velocity="2.0944"/>
+			<origin xyz="0 0.163 0" rpy="0 0 0"/>
+			<parent link="${prefix}shoulder"/>
+			<child link="${prefix}shoulder_roll_link"/>
 			<dynamics damping="0.7" friction="0.0"/>
 		</joint>
 		<transmission name="${prefix}tran2">
 			<type>transmission_interface/SimpleTransmission</type>
-			<joint name="${prefix}joint2">
+			<joint name="${prefix}shoulder_roll">
 				<hardwareInterface>EffortJointInterface</hardwareInterface>
 			</joint>
@@ -114,43 +83,43 @@
 			</actuator>
 		</transmission>
-		<link name="${prefix}link2b">
-			<collision>
-				<origin xyz="0 0 0" rpy="0 0 0"/>
-				<geometry>
-					<mesh filename="package://hdt_7dof_description/meshes/hdt_7dof_2b.STL"/>
-				</geometry>
-			</collision>
-			<visual>
-				<origin xyz="0 0 0.0" rpy="0 0 0"/>
-				<geometry>
-					<mesh filename="package://hdt_7dof_description/meshes/hdt_7dof_2b.STL"/>
-				</geometry>
-				<material name="${prefix}grey"/>
-			</visual>
-			<inertial>
-				<origin xyz="0 0 -0.02018105" rpy="0 0 0"/>
-				<mass value="0.69896"/>
-				<inertia
-				ixx="0.00088116" ixy="0.0" ixz="0.0"
-				iyy="0.00094182" iyz="0.0"
-				izz="0.00032992"/>
-			</inertial>
-		</link>
-		<gazebo reference="${prefix}link2b">
-			<material>Gazebo/Grey</material>
-		</gazebo>
-		<!-- segment 3 -->
-		<joint name="${prefix}joint3" type="revolute">
+		<link name="${prefix}shoulder_roll_link">
+			<collision>
+				<origin xyz="-0.06 -0.297925 -1.04" rpy="0 0 0"/>
+				<geometry>
+					<mesh filename="package://hdt_7dof_description/meshes/ShoulderRollLeft.stl" scale="0.001 0.001 0.001"/>
+				</geometry>
+			</collision>
+			<visual>
+				<origin xyz="-0.06 -0.297925 -1.04" rpy="0 0 0"/>
+				<geometry>
+					<mesh filename="package://hdt_7dof_description/meshes/ShoulderRollLeft.stl" scale="0.001 0.001 0.001"/>
+				</geometry>
+				<material name="${prefix}grey"/>
+			</visual>
+			<inertial>
+				<origin xyz="-0.000656538 -0.013605177 -0.015055902" rpy="0 0 0"/>
+				<mass value="0.709190454"/>
+				<inertia
+				ixx="0.006529967" ixy="-1.713e-06" ixz="-1.903e-06"
+				iyy="0.000866608" iyz="0.000532013"
+				izz="0.005955599"/>
+			</inertial>
+		</link>
+		<gazebo reference="${prefix}shoulder_roll_link">
+			<material>Gazebo/Grey</material>
+		</gazebo>
+		<!-- upper arm -->
+		<joint name="${prefix}shoulder_yaw" type="revolute">
 			<hdt id="43" kmin="75" kmax="150" inertia="0.075"/>
 			<axis xyz="0 0 1"/>
-			<limit effort="60.0" lower="-2.0944" upper="2.0944" velocity="2.0944"/>
-			<origin xyz="0 0 -0.077" rpy="0 0 0" />
-			<parent link="${prefix}link2b"/>
-			<child link="${prefix}link3"/>
+			<limit effort="60.0" lower="-2.0943951023932" upper="2.0943951023932" velocity="2.0944"/>
+			<origin xyz="0 0 0" rpy="0 0 0" />
+			<parent link="${prefix}shoulder_roll_link"/>
+			<child link="${prefix}arm"/>
 			<dynamics damping="0.7" friction="0.0"/>
 		</joint>
 		<transmission name="${prefix}tran3">
 			<type>transmission_interface/SimpleTransmission</type>
-			<joint name="${prefix}joint3">
+			<joint name="${prefix}shoulder_yaw">
 				<hardwareInterface>EffortJointInterface</hardwareInterface>
 			</joint>
@@ -159,74 +128,43 @@
 			</actuator>
 		</transmission>
-		<link name="${prefix}link3">
-			<collision>
-				<origin xyz="0 0 0.0" rpy="0 0 0"/>
-				<geometry>
-					<mesh filename="package://hdt_7dof_description/meshes/hdt_7dof_3.STL"/>
-				</geometry>
-			</collision>
-			<visual>
-				<origin xyz="0 0 0.0" rpy="0 0 0"/>
-				<geometry>
-					<mesh filename="package://hdt_7dof_description/meshes/hdt_7dof_3.STL"/>
+		<link name="${prefix}arm">
+			<collision>
+				<origin xyz="-0.06 -0.297925 -1.04" rpy="0 0 0"/>
+				<geometry>
+					<mesh filename="package://hdt_7dof_description/meshes/ShoulderYawLeft.stl" scale="0.001 0.001 0.001"/>
+				</geometry>
+			</collision>
+			<visual>
+				<origin xyz="-0.06 -0.297925 -1.04" rpy="0 0 0"/>
+				<geometry>
+					<mesh filename="package://hdt_7dof_description/meshes/ShoulderYawLeft.stl" scale="0.001 0.001 0.001"/>
 				</geometry>
 				<material name="${prefix}green"/>
 			</visual>
 			<inertial>
-				<origin xyz="0 0 -0.08013953" rpy="0 0 0"/>
-				<mass value="1.77733729"/>
-				<inertia
-				ixx="0.00450640" ixy="0.0" ixz="0.0"
-				iyy="0.00450640" iyz="0.0"
-				izz="0.00114447"/>
-			</inertial>
-		</link>
-		<gazebo reference="${prefix}link3">
+				<origin xyz="-0.000500004 0.00094170500000001 -0.209152474" rpy="0 0 0"/>
+				<mass value="1.291829307"/>
+				<inertia
+				ixx="0.007190942" ixy="-0" ixz="-0"
+				iyy="0.007116565" iyz="-0.000130703"
+				izz="0.000965322"/>
+			</inertial>
+		</link>
+		<gazebo reference="${prefix}arm">
 			<material>Gazebo/Green</material>
 		</gazebo>
-		<joint name="${prefix}joint3f" type="fixed">
-			<origin xyz="0 0 -0.16271" rpy="0 0 0"/>
-			<parent link="${prefix}link3"/>
-			<child link="${prefix}link4a"/>
-		</joint>
-		<link name="${prefix}link4a">
-			<collision>
-				<origin xyz="0 0 0" rpy="0 0 0"/>
-				<geometry>
-					<mesh filename="package://hdt_7dof_description/meshes/hdt_7dof_4a.STL"/>
-				</geometry>
-			</collision>
-			<visual>
-				<origin xyz="0 0 0.0" rpy="0 0 0"/>
-				<geometry>
-					<mesh filename="package://hdt_7dof_description/meshes/hdt_7dof_4a.STL"/>
-				</geometry>
-				<material name="${prefix}black"/>
-			</visual>
-			<inertial>
-				<origin xyz="0 0 -0.04416876" rpy="0 0 0"/>
-				<mass value="0.66774822"/>
-				<inertia
-				ixx="0.00091291" ixy="0.0" ixz="0.0"
-				iyy="0.00110241" iyz="0.0"
-				izz="0.00062987"/>
-			</inertial>
-		</link>
-		<gazebo reference="${prefix}link4a">
-			<material>Gazebo/Black</material>
-		</gazebo>
-		<!-- segment 4 -->
-		<joint name="${prefix}joint4" type="revolute">
+		<!-- elbow pitch -->
+		<joint name="${prefix}elbow_pitch" type="revolute">
 			<hdt id="44" kmin="75" kmax="150" inertia="0.075"/>
-			<axis xyz="-1 0 0"/>
-			<limit effort="60.0" lower="-0.5236" upper="3.6652" velocity="2.0944"/>
-			<origin xyz="0 0 -0.07" rpy="3.1416 0 0"/>
-			<parent link="${prefix}link4a"/>
-			<child link="${prefix}link4b"/>
+			<axis xyz="0 1 0"/>
+			<limit effort="60.0" lower="-3.6651914291881" upper="0.5235987755983" velocity="2.0944"/>
+			<origin xyz="0 0 -0.3186" rpy="0 0 0"/>
+			<parent link="${prefix}arm"/>
+			<child link="${prefix}elbow_link"/>
 			<dynamics damping="0.7" friction="0.0"/>
 		</joint>
 		<transmission name="${prefix}tran4">
 			<type>transmission_interface/SimpleTransmission</type>
-			<joint name="${prefix}joint4">
+			<joint name="${prefix}elbow_pitch">
 				<hardwareInterface>EffortJointInterface</hardwareInterface>
 			</joint>
@@ -235,119 +173,88 @@
 			</actuator>
 		</transmission>
-		<link name="${prefix}link4b">
-			<collision>
-				<origin xyz="0 0 0" rpy="0 0 0"/>
-				<geometry>
-					<mesh filename="package://hdt_7dof_description/meshes/hdt_7dof_4b.STL"/>
-				</geometry>
-			</collision>
-			<visual>
-				<origin xyz="0 0 0.0" rpy="0 0 0"/>
-				<geometry>
-					<mesh filename="package://hdt_7dof_description/meshes/hdt_7dof_4b.STL"/>
-				</geometry>
-				<material name="${prefix}grey"/>
-			</visual>
-			<inertial>
-				<origin xyz="0 -0.02018105 0" rpy="0 0 0"/>
-				<mass value="0.69896279"/>
-				<inertia
-				ixx="0.00094182" ixy="0.0" ixz="0.0"
-				iyy="0.00032992" iyz="0.0"
-				izz="0.00088116"/>
-			</inertial>
-		</link>
-		<gazebo reference="${prefix}link4b">
-			<material>Gazebo/Grey</material>
-		</gazebo>
-		<!-- segment 5 -->
-		<joint name="${prefix}joint5" type="revolute">
+		<link name="${prefix}elbow_link">
+			<collision>
+				<origin xyz="-0.06 -0.297925 -0.7214" rpy="0 0 0"/>
+				<geometry>
+					<mesh filename="package://hdt_7dof_description/meshes/ElbowLeft.stl" scale="0.001 0.001 0.001"/>
+				</geometry>
+			</collision>
+			<visual>
+				<origin xyz="-0.06 -0.297925 -0.7214" rpy="0 0 0"/>
+				<geometry>
+					<mesh filename="package://hdt_7dof_description/meshes/ElbowLeft.stl" scale="0.001 0.001 0.001"/>
+				</geometry>
+				<material name="${prefix}grey"/>
+			</visual>
+			<inertial>
+				<origin xyz="0.014260471 0.00015822900000001 -7.5344000000088e-05" rpy="0 0 0"/>
+				<mass value="0.923870693"/>
+				<inertia
+				ixx="0.000477001" ixy="-2.405e-06" ixz="-4.205e-06"
+				iyy="0.001214959" iyz="1.1e-08"
+				izz="0.001118907"/>
+			</inertial>
+		</link>
+		<gazebo reference="${prefix}elbow_link">
+			<material>Gazebo/Grey</material>
+		</gazebo>
+		<!-- forearm -->
+		<joint name="${prefix}elbow_yaw" type="revolute">
 			<hdt id="45" kmin="50" kmax="100" inertia="0.05"/>
-			<axis xyz="0 -1 0"/>
-			<limit effort="60.0" lower="-2.0944" upper="2.0944" velocity="2.0944"/>
-			<origin xyz="0 -0.077 0" rpy="0 3.1416 0"/>
-			<parent link="${prefix}link4b"/>
-			<child link="${prefix}link5"/>
+			<axis xyz="1 0 0"/>
+			<limit effort="60.0" lower="-2.0943951023932" upper="2.0943951023932" velocity="2.0944"/>
+			<origin xyz="0 0 0" rpy="0 0 0"/>
+			<parent link="${prefix}elbow_link"/>
+			<child link="${prefix}forearm"/>
 			<dynamics damping="0.7" friction="0.0"/>
 		</joint>
 		<transmission name="${prefix}tran5">
 			<type>transmission_interface/SimpleTransmission</type>
-			<joint name="${prefix}joint5">
-				<hardwareInterface>EffortJointInterface</hardwareInterface>
-			</joint>
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
File: urdf/hdt_7dof_right.xacro (robot description, xacro)
@@ -9,4 +9,4 @@
 	<link name="world" />
 	<xacro:include filename="$(find hdt_7dof_description)/urdf/hdt_7dof_right_macro.xacro" />
-	<xacro:hdt_7dof_right parent="world" x="0" y="0" z="0" yaw="1.57079" prefix="right_" />
+	<xacro:hdt_7dof_right parent="world" x="0" y="0" z="0" prefix="right_" />
 </robot>
